Commit message: add gitignore

File: ur_simplified_description/urdf/ur10e.urdf.xacro (robot description, xacro)
@@ -53,5 +53,5 @@
     <xacro:property name="base_correction" value="${pi}" />
     <link name="${prefix}base_link" >
-      <visual>
+      <!-- put with shoulder_link <visual>
         <origin xyz="0 0 0" rpy="0 0 ${base_correction}"/>
         <geometry>
@@ -67,5 +67,5 @@
           <cylinder length="0.1" radius="0.1"/>
         </geometry>
-      </collision>
+      </collision>-->
       <xacro:cylinder_inertial radius="0.075" length="0.038" mass="${base_mass}">
         <origin xyz="0.0 0.0 0.0" rpy="0 0 0" />
@@ -102,7 +102,7 @@
       </visual>
       <collision>
-        <origin xyz="0 0 0" rpy="0 0 0"/>
-        <geometry>
-          <cylinder length="0.20" radius="0.1"/>
+        <origin xyz="0 0 -0.05" rpy="0 0 0"/>
+        <geometry>
+          <cylinder length="0.30" radius="0.1"/>
         </geometry>
       </collision>

Commit message: base visual fixed

File: ur_simplified_description/urdf/ur10e.urdf.xacro (robot description, xacro)
@@ -53,5 +53,5 @@
     <xacro:property name="base_correction" value="${pi}" />
     <link name="${prefix}base_link" >
-      <!-- put with shoulder_link <visual>
+      <visual>
         <origin xyz="0 0 0" rpy="0 0 ${base_correction}"/>
         <geometry>
@@ -62,5 +62,5 @@
         </material>
       </visual>
-      <collision>
+     <!-- <collision>
         <origin xyz="0 0 0.05" rpy="0 0 0"/>
         <geometry>

Commit message: transition to new ur format

File: ur_simplified_description/urdf/ur10e.urdf.xacro (robot description, xacro)
@@ -5,6 +5,6 @@
   Contributers: Jimmy Da Silva, Ajit Krisshna N L, Muhammad Asif Rana
 -->
-  <xacro:include filename="$(find ur_e_description)/urdf/ur.transmission.xacro" />
-  <xacro:include filename="$(find ur_e_description)/urdf/ur.gazebo.xacro" />
+<xacro:include filename="$(find ur_description)/urdf/inc/ur_transmissions.xacro" />
+<xacro:include filename="$(find ur_description)/urdf/inc/ur_common.xacro" />
   <xacro:macro name="cylinder_inertial" params="radius length mass *origin">
     <inertial>
@@ -56,5 +56,5 @@
         <origin xyz="0 0 0" rpy="0 0 ${base_correction}"/>
         <geometry>
-          <mesh filename="package://ur_e_description/meshes/ur10e/visual/base.dae"/>
+          <mesh filename="package://ur_description/meshes/ur10e/visual/base.dae"/>
         </geometry>
         <material name="LightGrey">
@@ -95,5 +95,5 @@
         <origin xyz="0 0 0" rpy="0 0 ${pi}"/>
         <geometry>
-          <mesh filename="package://ur_e_description/meshes/ur10e/visual/shoulder.dae"/>
+          <mesh filename="package://ur_description/meshes/ur10e/visual/shoulder.dae"/>
         </geometry>
         <material name="LightGrey">
@@ -134,5 +134,5 @@
         <origin xyz="0 0 ${shoulder_offset}" rpy="${pi/2} 0 ${-pi/2}"/>
         <geometry>
-          <mesh filename="package://ur_e_description/meshes/ur10e/visual/upperarm.dae"/>
+          <mesh filename="package://ur_description/meshes/ur10e/visual/upperarm.dae"/>
         </geometry>
         <material name="LightGrey">
@@ -173,5 +173,5 @@
         <origin xyz="0 0 ${elbow_offset}" rpy="${pi/2} 0 ${-pi/2}"/>
         <geometry>
-          <mesh filename="package://ur_e_description/meshes/ur10e/visual/forearm.dae"/>
+          <mesh filename="package://ur_description/meshes/ur10e/visual/forearm.dae"/>
         </geometry>
         <material name="LightGrey">
@@ -212,5 +212,5 @@
         <origin xyz="0 0 -0.135" rpy="${pi/2} 0 0"/>
         <geometry>
-          <mesh filename="package://ur_e_description/meshes/ur10e/visual/wrist1.dae"/>
+          <mesh filename="package://ur_description/meshes/ur10e/visual/wrist1.dae"/>
         </geometry>
         <material name="LightGrey">
@@ -251,5 +251,5 @@
         <origin xyz="0 0 -0.12" rpy="0 0 0"/>
         <geometry>
-          <mesh filename="package://ur_e_description/meshes/ur10e/visual/wrist2.dae"/>
+          <mesh filename="package://ur_description/meshes/ur10e/visual/wrist2.dae"/>
         </geometry>
         <material name="LightGrey">
@@ -290,5 +290,5 @@
         <origin xyz="0 0 -0.1168" rpy="${pi/2} 0 0"/>
         <geometry>
-          <mesh filename="package://ur_e_description/meshes/ur10e/visual/wrist3.dae"/>
+          <mesh filename="package://ur_description/meshes/ur10e/visual/wrist3.dae"/>
         </geometry>
         <material name="LightGrey">
@@ -320,5 +320,4 @@
     </link>
     <xacro:ur_arm_transmission prefix="${prefix}" hw_interface="${transmission_hw_interface}" />
-    <xacro:ur_arm_gazebo prefix="${prefix}" />
     <!-- ROS base_link to UR 'Base' Coordinates transform -->
     <link name="${prefix}base"/>

File: ur_simplified_description/urdf/ur10e_robot.urdf.xacro (robot description, xacro)
@@ -2,9 +2,9 @@
 <robot xmlns:xacro="http://ros.org/wiki/xacro" name="ur10e" >
   <!-- common stuff -->
-  <xacro:include filename="$(find ur_e_description)/urdf/common.gazebo.xacro" />
+  <xacro:include filename="$(find ur_description)/urdf/common.gazebo.xacro" />
   <!-- ur10e -->
   <xacro:include filename="$(find ur_simplified_description)/urdf/ur10e.urdf.xacro" />
   <!-- arm -->
-  <xacro:arg name="kinematics_config" default="$(find ur_e_description)/config/ur10e_default.yaml"/>
+  <xacro:arg name="kinematics_config" default="$(find ur_description)/config/ur10e_default.yaml"/>
   <xacro:ur10e_robot prefix="" joint_limited="false"
     kinematics_file="${load_yaml('$(arg kinematics_config)')}"

Commit message: no collisions

File: ur_simplified_description/urdf/ur10e.urdf.xacro (robot description, xacro)
@@ -62,10 +62,7 @@
         </material>
       </visual>
-     <!-- <collision>
-        <origin xyz="0 0 0.05" rpy="0 0 0"/>
-        <geometry>
-          <cylinder length="0.1" radius="0.1"/>
-        </geometry>
-      </collision>-->
+      <collision>
+            <!--   NO COLLISIONS  -->
+      </collision>
       <xacro:cylinder_inertial radius="0.075" length="0.038" mass="${base_mass}">
         <origin xyz="0.0 0.0 0.0" rpy="0 0 0" />
@@ -318,4 +315,7 @@
         <origin rpy="0 0 0" xyz="-0.01 0 0"/>
       </visual>
+      <collision>
+            <!--   NO COLLISIONS  -->
+      </collision>
     </link>
     <xacro:ur_arm_transmission prefix="${prefix}" hw_interface="${transmission_hw_interface}" />

Commit message: fix

File: ur_simplified_description/urdf/ur10e.urdf.xacro (robot description, xacro)
@@ -63,5 +63,7 @@
       </visual>
       <collision>
-            <!--   NO COLLISIONS  -->
+        <geometry>
+            <cylinder length="0.0" radius="0.0"/>          <!--   NO COLLISIONS  -->
+        </geometry>
       </collision>
       <xacro:cylinder_inertial radius="0.075" length="0.038" mass="${base_mass}">
@@ -316,5 +318,7 @@
       </visual>
       <collision>
-            <!--   NO COLLISIONS  -->
+        <geometry>
+            <cylinder length="0.0" radius="0.0"/>          <!--   NO COLLISIONS  -->
+        </geometry>
       </collision>
     </link>
